Commit message: odomを追加

File: src/nhk24_use_amcl/urdf/description.urdf (robot description, URDF)
Before this commit: robot nhk24zero, 7 links, 6 joints
Links:
- added link odom
Joints:
- added joint odom_joint: type fixed, parent imu_link, child odom, origin xyz=0 0 0

File: src/nhk24_use_amcl/urdf/description.xacro (robot description, xacro)
@@ -157,4 +157,10 @@
 		</sensor>
 	</gazebo>
+	<link name="odom"></link>
+	<joint name="odom_joint" type="fixed">
+		<parent link="imu_link" />
+		<child link="odom" />
+		<origin xyz="0 0 0" />
+	</joint>
 	<link name="lidar_link">
 		<inertial>

Commit message: やっぱodomいらなくないか

File: src/nhk24_use_amcl/urdf/description.urdf (robot description, URDF)
Before this commit: robot nhk24zero, 8 links, 7 joints
Links:
- removed link odom
Joints:
- removed joint odom_joint

File: src/nhk24_use_amcl/urdf/description.xacro (robot description, xacro)
@@ -157,10 +157,4 @@
 		</sensor>
 	</gazebo>
-	<link name="odom"></link>
-	<joint name="odom_joint" type="fixed">
-		<parent link="imu_link" />
-		<child link="odom" />
-		<origin xyz="0 0 0" />
-	</joint>
 	<link name="lidar_link">
 		<inertial>

Commit message: emcl2はtfフレームのbase_footprintまで見ている。なんで？

File: src/nhk24_use_amcl/urdf/description.urdf (robot description, URDF)
Before this commit: robot nhk24zero, 7 links, 6 joints
Links:
- added link base_footprint_link
Joints:
- added joint base_footprint_joint: type fixed, parent base_link, child base_footprint_link, origin xyz=0 0 0

File: src/nhk24_use_amcl/urdf/description.xacro (robot description, xacro)
@@ -39,4 +39,11 @@
 		<xacro:box_inertia m="15" w="${base_width}" d="${base_length}" h="${base_height}"/>
 	</link>
+	<link name="base_footprint_link">
+	</link>
+	<joint name="base_footprint_joint" type="fixed">
+		<parent link="base_link" />
+		<child link="base_footprint_link" />
+		<origin xyz="0 0 0" />
+	</joint>
 	<!-- Omni Wheels -->
 	<xacro:macro name="wheel" params="prefix x_reflect y_reflect wheel_yaw">

Commit message: Lidar取り付け位置の変更

File: src/nhk24_use_amcl/urdf/description.urdf (robot description, URDF)
Before this commit: robot nhk24zero, 8 links, 7 joints
Joints:
- joint lidar_joint: origin xyz=0 0 0 rpy=0 0 0 -> xyz=0.10 -0.40 0.13 rpy=1.5707963267948966 0 -1.5707963267948966

File: src/nhk24_use_amcl/urdf/description.xacro (robot description, xacro)
@@ -186,5 +186,5 @@
 		<parent link="base_link"/>
 		<child link="lidar_link"/>
-		<origin xyz="0 0 0" rpy="0 0 0"/>
+		<origin xyz="0.10 -0.40 0.13" rpy="${pi/2} 0 ${-pi/2}"/>
 	  </joint>
 	  <gazebo reference="lidar_link">

Commit message: lidar_linkを修正

File: src/nhk24_use_amcl/urdf/description.urdf (robot description, URDF)
Before this commit: robot nhk24zero, 8 links, 7 joints
Joints:
- joint lidar_joint: origin xyz=0.10 -0.40 0.13 rpy=1.5707963267948966 0 -1.5707963267948966 -> xyz=0.10 -0.40 0.13 rpy=3.141592653589793 0 -1.5707963267948966

File: src/nhk24_use_amcl/urdf/description.xacro (robot description, xacro)
@@ -186,5 +186,5 @@
 		<parent link="base_link"/>
 		<child link="lidar_link"/>
-		<origin xyz="0.10 -0.40 0.13" rpy="${pi/2} 0 ${-pi/2}"/>
+		<origin xyz="0.10 -0.40 0.13" rpy="${pi} 0 ${-pi/2}"/>
 	  </joint>
 	  <gazebo reference="lidar_link">

Commit message: 椅子載せ機体用

File: src/nhk24_use_amcl/urdf/description.urdf (robot description, URDF)
Before this commit: robot nhk24zero, 8 links, 7 joints
Joints:
- joint lidar_joint: origin xyz=0.10 -0.40 0.13 rpy=3.141592653589793 0 -1.5707963267948966 -> xyz=0.25 0 0.70 rpy=0 0 0

File: src/nhk24_use_amcl/urdf/description.xacro (robot description, xacro)
@@ -186,5 +186,5 @@
 		<parent link="base_link"/>
 		<child link="lidar_link"/>
-		<origin xyz="0.10 -0.40 0.13" rpy="${pi} 0 ${-pi/2}"/>
+		<origin xyz="0.25 0 0.70" rpy="0 0 0"/>
 	  </joint>
 	  <gazebo reference="lidar_link">

Commit message: あたらしいテスト機体に合わせた

File: src/nhk24_use_amcl/urdf/description.urdf (robot description, URDF)
Before this commit: robot nhk24zero, 8 links, 7 joints
Joints:
- joint lidar_joint: origin xyz=0.25 0 0.70 rpy=0 0 0 -> xyz=0 0 0.70 rpy=0 0 3.141592653589793

File: src/nhk24_use_amcl/urdf/description.xacro (robot description, xacro)
@@ -186,5 +186,5 @@
 		<parent link="base_link"/>
 		<child link="lidar_link"/>
-		<origin xyz="0.25 0 0.70" rpy="0 0 0"/>
+		<origin xyz="0 0 0.70" rpy="0 0 ${pi}"/>
 	  </joint>
 	  <gazebo reference="lidar_link">
