Commit message: ライダーのjointを変更

File: urdf/description.urdf (robot description, URDF)
Before this commit: robot nhk24zero, 8 links, 7 joints
Joints:
- joint lidar_joint: origin xyz=0 0 0.70 rpy=0 0 3.141592653589793 -> xyz=0 -0.250 0.015 rpy=0 3.141592653589793 3.141592653589793/2

File: urdf/description.xacro (robot description, xacro)
@@ -186,5 +186,5 @@
 		<parent link="base_link"/>
 		<child link="lidar_link"/>
-		<origin xyz="0 0 0.70" rpy="0 0 ${pi}"/>
+		<origin xyz="0 -0.250 0.015" rpy="0 ${pi} ${pi}/2"/>
 	  </joint>
 	  <gazebo reference="lidar_link">

Commit message: テスト機体用に

File: urdf/description.urdf (robot description, URDF)
Before this commit: robot nhk24zero, 8 links, 7 joints
Links:
- added link camera_link; visual box size=0.1 0.1 0.1
Joints:
- added joint camera_joint: type fixed, parent base_link, child camera_link, origin xyz=0 0.500 0.200 rpy=-1.5707963267948966 0 0
- joint lidar_joint: origin xyz=0 -0.250 0.015 rpy=0 3.141592653589793 3.141592653589793/2 -> xyz=0 -0 0.0200 rpy=0 0 0

File: urdf/description.xacro (robot description, xacro)
@@ -182,11 +182,11 @@
 		  </geometry>
 		</visual>
-	  </link>
-	  <joint name="lidar_joint" type="fixed">
+	</link>
+	<joint name="lidar_joint" type="fixed">
 		<parent link="base_link"/>
 		<child link="lidar_link"/>
-		<origin xyz="0 -0.250 0.015" rpy="0 ${pi} ${pi}/2"/>
-	  </joint>
-	  <gazebo reference="lidar_link">
+		<origin xyz="0 -0 0.0200" rpy="0 0 0"/>
+	</joint>
+	<gazebo reference="lidar_link">
 		<sensor name="lidar" type="ray">
 		  <always_on>true</always_on>
@@ -222,3 +222,15 @@
 		</sensor>
 	  </gazebo>
+	<link name="camera_link">
+		<visual>
+			<geometry>
+				<box size="0.1 0.1 0.1" />
+			</geometry>
+		</visual>
+	</link>
+	<joint name="camera_joint" type="fixed">
+		<parent link="base_link"/>
+		<child link="camera_link"/>
+		<origin xyz="0 0.500 0.200" rpy="${-pi/2} 0 0"/>
+	</joint>
 </robot>

Commit message: どうも、urdfのjointのoriginのrpyはy, p, rの順に回るらしい？

File: urdf/description.urdf (robot description, URDF)
Before this commit: robot nhk24zero, 8 links, 7 joints
Joints:
- joint lidar_joint: origin xyz=0 -0.250 0.015 rpy=0 3.141592653589793 3.141592653589793/2 -> xyz=0 0 0.3 rpy=0 0 0

File: urdf/description.xacro (robot description, xacro)
@@ -186,5 +186,6 @@
 		<parent link="base_link"/>
 		<child link="lidar_link"/>
-		<origin xyz="0 -0.250 0.015" rpy="0 ${pi} ${pi}/2"/>
+		<!-- <origin xyz="-0.250 0 0.015" rpy="0 ${pi} 0"/> -->
+		<origin xyz="0 0 0.3" rpy="0 0 0"/>
 	  </joint>
 	  <gazebo reference="lidar_link">
